File: switch_breakout.kicad_pcb (KiCad board)
At the start: 2 copper layers, 22 x 15 mm, 2 parts, among them J1 Switch, SW1 SW_DPDT

Commit message: Prepare release of 1.0.1
Other:
- board text added: "Switch breakout board 11/23 Rev 1.0.1"
- board text removed: "Switch breakout board 06/23 Rev 1.0"
Changed lines of the file:
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@@
   (gr_line (start 137 94) (end 137 81)
     (stroke (width 0.1) (type solid)) (layer "Edge.Cuts"))
-  (gr_text "Switch breakout board\n06/23 Rev 1.0" (at 136 81.7) (layer "B.SilkS")
+  (gr_text "Switch breakout board\n11/23 Rev 1.0.1" (at 136 81.7) (layer "B.SilkS")
     (effects (font (size 1 1) (thickness 0.15)) (justify left mirror))
   )
